File: filtro_PB_4to_L-R.kicad_sch (KiCad schematic)
At the start: 20 parts, among them J1 Conn_01x03, J2 Conn_01x03, J3 Conn_01x03, U1 NE5532

Commit message: Fix J2 and J3 connector values
Parts:
- J2, J3: value Conn_01x03 -> Conn_01x02
Changed lines of the file:
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@@
 			)
 		)
-		(property "Value" "Conn_01x03"
+		(property "Value" "Conn_01x02"
 			(at 53.34 83.82 0)
 			(effects
@@
 			)
 		)
-		(property "Value" "Conn_01x03"
+		(property "Value" "Conn_01x02"
 			(at 236.22 78.74 0)
 			(effects
